File: parts/add/add.kicad_pcb (KiCad board)
At the start: 2 copper layers, 70.6 x 106.7 mm, 31 parts, among them J1 Conn_02x02_Odd_Even, J2 Conn_01x02, J3 Conn_02x04_Odd_Even, J4 Conn_02x04_Odd_Even, J5 Conn_02x04_Odd_Even, J6 Conn_02x04_Odd_Even, J7 Conn_01x02, K1 HK19F, K10 HK19F, K11 HK19F, K12 HK19F, K13 HK19F, K14 HK19F, K15 HK19F, K16 HK19F, K2 HK19F, K3 HK19F, K4 HK19F, K5 HK19F, K6 HK19F, K7 HK19F, K8 HK19F, K9 HK19F

Commit message: Commit everything before the new KiCad eats my schematics.
Parts:
- removed J1: Conn_02x02_Odd_Even, Pin_Headers:Pin_Header_Straight_2x02_Pitch2.54mm
Other:
- board text added: "1"
- board text added: "A+B"
- board text added: "CARRY IN"
- board text added: "CARRY OUT"
- board text added: "IN A"
- board text added: "IN B"
- board text added: "IN ~A"
- board text added: "~CARRY IN"
- board text added: "~CARRY OUT"

Commit message: Update to new Kicad, finish reg.
Changed lines of the file:
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@@
-(kicad_pcb (version 4) (host pcbnew 4.0.7)
+(kicad_pcb (version 20171130) (host pcbnew 5.0.1)
   (general
-    (links 106)
-    (no_connects 0)
-    (area 103.581999 40.589999 174.294001 147.370001)
     (thickness 1.6)
     (drawings 18)
@@
   (page A4)
   (layers
-    (0 F.Cu signal)
-    (31 B.Cu signal)
+    (0 F.Cu signal hide)
+    (31 B.Cu signal hide)
     (32 B.Adhes user)
     (33 F.Adhes user)
@@
     (47 F.CrtYd user)
     (48 B.Fab user)
-    (49 F.Fab user)
+    (49 F.Fab user hide)
   )
   (setup
@@
     (pad_drill 0.6)
     (pad_to_mask_clearance 0.0508)
+    (solder_mask_min_width 0.25)
     (aux_axis_origin 0 0)
     (visible_elements FFFFFFFF)
@@
       (layerselection 0x00030_80000001)
       (usegerberextensions false)
+      (usegerberattributes false)
+      (usegerberadvancedattributes false)
+      (creategerberjobfile false)
       (excludeedgelayer true)
       (linewidth 0.100000)
@@
       (hpglpennumber 1)
       (hpglpenspeed 20)
-      (hpglpendiameter 15)
-      (hpglpenoverlay 2)
+      (hpglpendiameter 15.000000)
       (psnegative false)
       (psa4output false)
@@
     (effects (font (size 1.5 1.5) (thickness 0.3)))
   )
-  (gr_text "~CARRY IN" (at 112.268 49.784 90) (layer F.SilkS)
+  (gr_text "~CARRY IN" (at 112.268 49.784 270) (layer F.SilkS)
     (effects (font (size 1.5 1.5) (thickness 0.3)))
   )
-  (gr_text "CARRY IN" (at 109.728 49.784 90) (layer F.SilkS)
+  (gr_text "CARRY IN" (at 109.728 49.784 270) (layer F.SilkS)
     (effects (font (size 1.5 1.5) (thickness 0.3)))
   )
