File: parts/reg/reg.sch (KiCad schematic (older format))
At the start: 53 parts, among them J1 Conn_02x02_Odd_Even, J2 Conn_02x04_Odd_Even, J3 Conn_02x04_Odd_Even, J4 Conn_01x02, J5 Conn_02x04_Odd_Even, K1 HK19F, K10 HK19F, K11 HK19F, K12 HK19F, K2 HK19F, K3 HK19F, K4 HK19F, K5 HK19F, K6 HK19F, K7 HK19F, K8 HK19F, K9 HK19F

Commit message: Update to new Kicad, finish reg.
Parts:
- added J6: Conn_02x04_Odd_Even, Pin_Headers:Pin_Header_Straight_2x04_Pitch2.54mm, symbol reg-rescue:Conn_02x04_Odd_Even
- C1, C2, C3, C4, C5, C6, C7, C8: symbol CP -> reg-rescue:CP
- D1, D10, D11, D12, D2, D3, D4, D5, D6, D7, D8, D9: symbol D -> reg-rescue:D
- J1: symbol Conn_02x02_Odd_Even -> reg-rescue:Conn_02x02_Odd_Even
- J2, J3, J5: symbol Conn_02x04_Odd_Even -> reg-rescue:Conn_02x04_Odd_Even
- J4: symbol Conn_01x02 -> reg-rescue:Conn_01x02
- K1, K10, K11, K12, K2, K3, K4, K5, K6, K7, K8, K9: symbol HK19F -> reg-rescue:HK19F
- R1, R10, R11, R12, R13, R14, R15, R16, R2, R3, R4, R5, R6, R7, R8, R9: symbol R -> reg-rescue:R
Connections:
- net at D1.1 (K), K1.1, K9.6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: now also J6.1 (Pin_1)
- net at D2.1 (K), K2.1, K9.11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: now also J6.2 (Pin_2)
- net at D3.1 (K), K10.6, K3.1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: now also J6.3 (Pin_3)
- net at D4.1 (K), K10.11, K4.1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: now also J6.4 (Pin_4)
- net at D5.1 (K), K11.6, K5.1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: now also J6.5 (Pin_5)
- net at D6.1 (K), K11.11, K6.1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: now also J6.6 (Pin_6)
- net at D7.1 (K), K12.6, K7.1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: now also J6.7 (Pin_7)
- net at D8.1 (K), K12.11, K8.1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: now also J6.8 (Pin_8)
Other:
- note added: "override"
- moved on the sheet: C1, C2, C3, C4, C5, C6, C7, C8, D10, D11, D12, D9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
