File: new-parts/template/template.kicad_pcb (KiCad board)
At the start: 2 copper layers, 101.6 x 101.6 mm, 4 parts, among them J1 BHR-10-VUA, J2 BHR-10-VUA, K1 J104D2C12VDC.15S

Commit message: template: import design rules.
Other:
- rule pad_to_mask_clearance: 0 -> 0.038
Changed lines of the file:
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@@
   )
   (setup
-    (pad_to_mask_clearance 0)
+    (pad_to_mask_clearance 0.038)
+    (solder_mask_min_width 0.1)
     (pcbplotparams
       (layerselection 0x00010fc_ffffffff)
@@
         (effects (font (size 1 1) (thickness 0.15)))
     )
-    (fp_text value "BHR-10-VUA" (at 1.27 16.26) (layer "F.Fab")
+    (fp_text value "BHR-10-VUA" (at 1.27 16.26) (layer "F.Fab") hide
         (effects (font (size 1 1) (thickness 0.15)))
     )
@@
         (effects (font (size 1 1) (thickness 0.15)))
     )
-    (fp_text value "SMAJ14CA" (at 0 2.6 90) (layer "F.Fab")
+    (fp_text value "SMAJ14CA" (at 0 2.6 90) (layer "F.Fab") hide
         (effects (font (size 1 1) (thickness 0.15)))
     )
@@
         (effects (font (size 1 1) (thickness 0.15)))
     )
-    (fp_text value "J104D2C12VDC.15S" (at 8.4 2.4) (layer "F.Fab")
+    (fp_text value "J104D2C12VDC.15S" (at 8.4 2.4) (layer "F.Fab") hide
         (effects (font (size 1 1) (thickness 0.15)))
     )
@@
         (effects (font (size 1 1) (thickness 0.15)))
     )
-    (fp_text value "BHR-10-VUA" (at 1.27 16.26) (layer "F.Fab")
-        (effects (font (size 1 1) (thickness 0.15)))
-    )
+    (fp_text value "BHR-10-VUA" (at 1.27 16.26) (layer "F.Fab") hide
+        (effects (font (size 1 1) (thickness 0.15)))
+    )
