File: new-parts/mem/mem.kicad_sch (KiCad schematic)
At the start: 20 parts, among them J1 BHR-10-VUA, J2 BHR-10-VUA, J3 Conn_01x02, J4 BHR-10-VUA, U1 STM32F042C6Tx, U2 DRV8908

Commit message: Finish mem schematics and most of its layout.
Parts:
- removed J2, J4: BHR-10-VUA, Connector_IDC:IDC-Header_2x05_P2.54mm_Vertical, symbol Connector_Generic:Conn_02x05_Odd_Even
- removed J3: Conn_01x02, Connector_PinHeader_2.54mm:PinHeader_2x01_P2.54mm_Vertical, symbol Connector_Generic:Conn_01x02
- added C14: 10u, Capacitor_THT:CP_Radial_D10.0mm_P5.00mm, symbol Device:C_Polarized
- added C15: 22u, Capacitor_SMD:C_0805_2012Metric_Pad1.18x1.45mm_HandSolder, symbol Device:C
- added J1: Conn_02x02_Odd_Even, Connector_PinHeader_2.54mm:PinHeader_2x02_P2.54mm_Vertical, symbol Connector_Generic:Conn_02x02_Odd_Even
- added J2, J7, J8: Conn_02x01, Connector_PinHeader_2.54mm:PinHeader_1x02_P2.54mm_Vertical, symbol Connector_Generic:Conn_02x01
- added J3: USB_C_Receptacle_USB2.0, Connector_USB:USB_C_Receptacle_GCT_USB4105-xx-A_16P_TopMnt_Horizontal, symbol Connector:USB_C_Receptacle_USB2.0
- added J4: Conn_01x06, Connector_PinHeader_2.54mm:PinHeader_1x06_P2.54mm_Vertical, symbol Connector_Generic:Conn_01x06
- added J5: BHR-10-VUA, Connector_IDC:IDC-Header_2x05_P2.54mm_Vertical, symbol Connector_Generic:Conn_02x05_Odd_Even
- added R10, R11, R12, R21, R22, R23, R24, R25, R26, R27, R28, R29, R30, R5, R6, R7, R8, R9: 10k, Resistor_SMD:R_0805_2012Metric_Pad1.20x1.40mm_HandSolder, symbol Device:R
- added R13, R14, R15, R16, R17, R18, R19, R20, R31, R32, R33, R34, R35, R36, R37, R38, R39, R40: 2.2k, Resistor_SMD:R_0805_2012Metric_Pad1.20x1.40mm_HandSolder, symbol Device:R
- added R2: 5.1k, Resistor_SMD:R_0805_2012Metric_Pad1.20x1.40mm_HandSolder, symbol Device:R
- added R3: 33k, Resistor_SMD:R_0805_2012Metric_Pad1.20x1.40mm_HandSolder, symbol Device:R
- added R4: 82k, Resistor_SMD:R_0805_2012Metric_Pad1.20x1.40mm_HandSolder, symbol Device:R
- added U3: AZ1117H2-3.3, Package_TO_SOT_SMD:SOT-223-3_TabPin2, symbol az1117ch2:AZ1117H2-3.3
- added U4: USBLC6-2SC6, Package_TO_SOT_SMD:SOT-23-6, symbol Power_Protection:USBLC6-2SC6
- added U5, U6, U7, U8, U9: LTV-247, Package_SO:SOP-16_4.4x10.4mm_P1.27mm, symbol Isolator:LTV-247
- C1: renamed from C7; footprint Capacitor_THT:CP_Radial_D10.0mm_P5.00mm -> Capacitor_SMD:C_0805_2012Metric_Pad1.18x1.45mm_HandSolder; symbol Device:C_Polarized -> Device:C
- C10: renamed from C11; footprint Capacitor_THT:CP_Radial_D10.0mm_P5.00mm -> Capacitor_SMD:C_0805_2012Metric_Pad1.18x1.45mm_HandSolder; symbol Device:C_Polarized -> Device:C
- C2: renamed from C6; footprint Capacitor_THT:CP_Radial_D10.0mm_P5.00mm -> Capacitor_SMD:C_0805_2012Metric_Pad1.18x1.45mm_HandSolder; symbol Device:C_Polarized -> Device:C
- C3: renamed from C5; footprint Capacitor_THT:CP_Radial_D10.0mm_P5.00mm -> Capacitor_SMD:C_0805_2012Metric_Pad1.18x1.45mm_HandSolder; symbol Device:C_Polarized -> Device:C
- C8: renamed from C13; footprint Capacitor_THT:CP_Radial_D10.0mm_P5.00mm -> Capacitor_SMD:C_0805_2012Metric_Pad1.18x1.45mm_HandSolder; symbol Device:C_Polarized -> Device:C
- C9: renamed from C12; footprint Capacitor_THT:CP_Radial_D10.0mm_P5.00mm -> Capacitor_SMD:C_0805_2012Metric_Pad1.18x1.45mm_HandSolder; symbol Device:C_Polarized -> Device:C
- R1: value 10k -> 5.1k
- renumbered C10 to C11, C9 to C12, C8 to C13, C3 to C5, C2 to C6, C1 to C7, J1 to J6
Connections:
- net +12V: now also C14.1, J1.1 (Pin_1), J1.3 (Pin_3), J5.9 (Pin_9), U3.1 (VI)
- net +3V3: now also U1.1 (VBAT), U2.8 (~{SLEEP}), C15.1, J4.6 (Pin_6), U3.3 (VO), U5.10, U5.12, U5.14, U5.16, U6.10, U6.12, U6.14, U6.16, U7.10, U7.12, U7.14, U7.16, U8.10, U8.12, U8.14, U8.16, U9.14, U9.16; no longer R1.1
- net GND: now also R1.2, U2.25 (GND), C14.2, C15.2, J1.2 (Pin_2), J1.4 (Pin_4), J2.2 (Pin_2), J3.A1 (GND), J3.A12 (GND), J3.B1 (GND), J3.B12 (GND), J3.S1 (SHIELD), J4.1 (Pin_1), J4.5 (Pin_5), J5.10 (Pin_10), J7.2 (Pin_2), J8.2 (Pin_2), R10.1, R11.1, R12.1, R2.2, R21.1, R22.1, R23.1, R24.1, R25.1, R26.1, R27.1, R28.1, R29.1, R30.1, R4.1, R5.1, R6.1, R7.1, R8.1, R9.1, U3.2 (GND), U4.2 (GND), U5.2, U5.4, U5.6, U5.8, U6.2, U6.4, U6.6, U6.8, U7.2, U7.4, U7.6, U7.8, U8.2, U8.4, U8.6, U8.8, U9.2, U9.4; no longer U2.8 (~{SLEEP})
- net a0: now also R21.2, U7.15
- net a1: now also R22.2, U7.13
- net a2: now also R23.2, U7.11
- net a3: now also R24.2, U7.9
- net a4: now also R25.2, U8.15
- net a5: now also R26.2, U8.13
- net a6: now also R27.2, U8.11
- net a7: now also R28.2, U8.9
- net clk: now also R29.2, U9.15
- net in0: now also R5.2, U5.9
- net in1: now also R6.2, U5.11
- net in2: now also R7.2, U5.13
- net in3: now also R8.2, U5.15
- net in4: now also R9.2, U6.9
- net in5: now also R10.2, U6.11
- net in6: now also R11.2, U6.13
- net in7: now also R12.2, U6.15
- net swdclk: now also J4.3 (Pin_3)
- net swdio: now also J4.4 (Pin_4)
- net w/~{r}: now also R30.2, U9.13
- net ~{rst}: now reaches U1.7 (NRST)
- net ~{rst}: now also J4.2 (Pin_2); no longer R1.2
- net out0: now reaches U2.2 (OUT1)
- net out0: now also J5.1 (Pin_1), R13.2
- net out1: now reaches U2.23 (OUT2)
- net out1: now also J5.2 (Pin_2), R14.2
- net out2: now reaches U2.14 (OUT3)
- net out2: now also J5.3 (Pin_3), R15.2
- net out3: now reaches U2.11 (OUT4)
- net out3: now also J5.4 (Pin_4), R16.2
- net out4: now reaches U2.3 (OUT5)
- net out4: now also J5.5 (Pin_5), R17.2
- net out5: now reaches U2.10 (OUT6)
- net out5: now also J5.6 (Pin_6), R18.2
- net out6: now reaches U2.4 (OUT7)
- net out6: now also J5.7 (Pin_7), R19.2
- net out7: now reaches U2.22 (OUT8)
- net out7: now also J5.8 (Pin_8), R20.2
- net at J6.1 (Pin_1): now also R31.2
- net at J6.2 (Pin_2): now also R32.2
- net at J6.3 (Pin_3): now also R33.2
- net at J6.4 (Pin_4): now also R34.2
- net at J6.5 (Pin_5): now also R35.2
- net at J6.6 (Pin_6): now also R36.2
- net at J6.7 (Pin_7): now also R37.2
- net at J6.8 (Pin_8): now also R38.2
- net vbus_sense: now reaches U1.31 (PA10)
- net vbus_sense: now also R3.1, R4.2
- net boot0: now reaches U1.44 (PF11)
- net boot0: now also J2.1 (Pin_1)
- net drv_fault renamed ~{fault}
- net usb_dm renamed usb_dN
- net usb_dN: now also U4.6 (I/O1)
- net usb_dp renamed usb_dP
- net usb_dP: now also U4.4 (I/O2)
- new net: R19.1, U6.3
- new net: R20.1, U6.1
- new net: R31.1, U7.1
- new net: R37.1, U8.5
- new net: R33.1, U7.5
- new net: R18.1, U6.5
- new net: R17.1, U6.7
- new net: R40.1, U9.3
- new net: R34.1, U7.7
- new net: R16.1, U5.1
- new net: R13.1, U5.7
- new net: R36.1, U8.3
- new net: J8.1 (Pin_1), R40.2
- new net: R39.1, U9.1
- new net: R38.1, U8.7
- new net: J7.1 (Pin_1), R39.2
- new net: J3.A4 (VBUS), J3.A9 (VBUS), J3.B4 (VBUS), J3.B9 (VBUS), R3.2, U4.5 (VBUS)
- new net: J3.A5 (CC1), R1.1
- new net: J3.B5 (CC2), R2.1
- new net: R32.1, U7.3
- new net: R14.1, U5.5
- new net: R35.1, U8.1
- new net: R15.1, U5.3
- new net usbplug_dN: J3.A7 (D-), J3.B7 (D-), U4.1 (I/O1)
- new net usbplug_dP: J3.A6 (D+), J3.B6 (D+), U4.3 (I/O2)
- no-connect marks 0 -> 10
Other:
- note added: "For divider spec see STM document AN4879, sec. 2.6"
- note added: "address in"
- note added: "boot mode"
- note added: "clk in"
- note added: "data in/out"
- note added: "power"
- note added: "reset/debug"
- note added: "w/~{r} in"
- moved on the sheet: C11, C12, C13, C4, C5, C6, C7, J6, U1
