File: new-parts/mem-esp/mem-esp.kicad_sch (KiCad schematic)
At the start: 62 parts, among them J1 Conn_02x02_Odd_Even, J2 BHR-10-VUA, J3 BHR-10-VUA, J4 Conn_02x01, J5 Conn_02x01, J6 Conn_02x01, J7 Conn_02x01, U1 MC78M06_TO252, U2 ESP32-S3-DevKitC, U3 LTV-247, U4 LTV-247, U5 DRV8908, U6 LTV-247, U7 LTV-247, U8 LTV-247

Commit message: Finish layouting mem-esp.
Parts:
- added R41: 10k, Resistor_SMD:R_0805_2012Metric_Pad1.20x1.40mm_HandSolder, symbol Device:R
Connections:
- net +3V3: now also R41.1
- net ~{fault}: now also R41.2
Changed lines of the file:
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@@
   (junction (at 273.05 77.47) (diameter 0) (color 0 0 0 0)
   )
+  (junction (at 283.21 184.15) (diameter 0) (color 0 0 0 0)
+  )
   (junction (at 247.65 162.56) (diameter 0) (color 0 0 0 0)
   )
@@
     (stroke (width 0) (type default))
   )
-  (wire (pts (xy 283.21 184.15) (xy 283.21 173.99))
+  (wire (pts (xy 283.21 173.99) (xy 283.21 184.15))
     (stroke (width 0) (type default))
   )
@@
     (stroke (width 0) (type default))
   )
+  (wire (pts (xy 293.37 184.15) (xy 295.91 184.15))
+    (stroke (width 0) (type default))
+  )
   (wire (pts (xy 231.14 134.62) (xy 218.44 134.62))
     (stroke (width 0) (type default))
@@
     (stroke (width 0) (type default))
   )
+  (wire (pts (xy 283.21 184.15) (xy 285.75 184.15))
+    (stroke (width 0) (type default))
+  )
   (wire (pts (xy 123.19 36.83) (xy 139.7 36.83))
     (stroke (width 0) (type default))
@@
     (stroke (width 0) (type default))
   )
+  (wire (pts (xy 283.21 184.15) (xy 283.21 195.58))
+    (stroke (width 0) (type default))
+  )
   (wire (pts (xy 341.63 180.34) (xy 328.93 180.34))
     (stroke (width 0) (type default))
@@
     (effects (font (size 1.27 1.27)) (justify left bottom))
   )
-  (label "~{fault}" (at 283.21 181.61 90) (fields_autoplaced)
+  (label "~{fault}" (at 283.21 193.04 90) (fields_autoplaced)
     (effects (font (size 1.27 1.27)) (justify left bottom))
   )
@@
     )
   )
+  (symbol (lib_id "Device:R") (at 289.56 184.15 270) (unit 1)
+    (in_bom yes) (on_board yes) (dnp no) (fields_autoplaced)
+    (property "Reference" "R41" (at 289.56 177.8 90)
+      (effects (font (size 1.27 1.27)))
+    )
+    (property "Value" "10k" (at 289.56 180.34 90)
+      (effects (font (size 1.27 1.27)))
+    )
+    (property "Footprint" "Resistor_SMD:R_0805_2012Metric_Pad1.20x1.40mm_HandSolder" (at 289.56 182.372 90)
+      (effects (font (size 1.27 1.27)) hide)
+    )
+    (property "Datasheet" "~" (at 289.56 184.15 0)
+      (effects (font (size 1.27 1.27)) hide)
+    )
+    (pin "1")
+    (pin "2")
+    (instances
+      (project "mem-esp"
+        (path "/8e7358e7-c3ef-4f3e-9154-e7eba01c544e"
+          (reference "R41") (unit 1)
+        )
+      )
+    )
+  )
   (symbol (lib_id "power:GND") (at 328.93 190.5 0) (unit 1)
     (in_bom yes) (on_board yes) (dnp no)
@@
         )
       )
+    )
+  )
+  (symbol (lib_id "power:+3V3") (at 295.91 184.15 270) (unit 1)
+    (in_bom yes) (on_board yes) (dnp no) (fields_autoplaced)
+    (property "Reference" "#PWR097" (at 292.1 184.15 0)
+      (effects (font (size 1.27 1.27)) hide)
+    )
+    (property "Value" "+3V3" (at 299.72 184.15 90)
+      (effects (font (size 1.27 1.27)) (justify left))
+    )
+    (property "Footprint" "" (at 295.91 184.15 0)
+      (effects (font (size 1.27 1.27)) hide)
+    )
+    (property "Datasheet" "" (at 295.91 184.15 0)
+      (effects (font (size 1.27 1.27)) hide)
+    )
+    (pin "1")
+    (instances
+      (project "mem-esp"
+        (path "/8e7358e7-c3ef-4f3e-9154-e7eba01c544e"
+          (reference "#PWR097") (unit 1)
+        )
+      )
