File: new-parts/mem-esp/mem-esp.kicad_pcb (KiCad board)
At the start: 2 copper layers, 134.6 x 49.5 mm, 70 parts, among them J1 Conn_02x02_Odd_Even, J2 BHR-10-VUA, J3 BHR-10-VUA, J4 Conn_01x01, J5 Conn_01x01, J6 Conn_01x01, J7 Conn_01x01, J8 BHR-10-VUA, U1 BA7806CP-E2, U2 ESP32-S3-DevKitC, U3 LTV-247, U4 LTV-247, U5 DRV8908, U6 LTV-247, U7 LTV-247, U8 LTV-247, U9 DRV8908

Commit message: Add signatures to some boards.
Other:
- board text added: "github.com/fread/visvitalis"
Changed lines of the file:
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@@
 		)
 		(pad_to_mask_clearance 0.038)
-		(solder_mask_min_width 0.1)
 		(allow_soldermask_bridges_in_footprints no)
 		(pcbplotparams
@@
 		)
 	)
+	(gr_text "github.com/fread/visvitalis"
+		(at 228.289777 116.050405 0)
+		(layer "B.SilkS")
+		(effects
+			(font
+				(size 1.5 1.5)
+				(thickness 0.3)
+				(bold yes)
+			)
+			(justify left mirror)
+		)
+	)
