File: new-parts/8mux/8mux.kicad_pcb (KiCad board)
At the start: 2 copper layers, 68.6 x 73.7 mm, 9 parts, among them J1 BHR-10-VUA, J2 BHR-10-VUA, J3 BHR-10-VUA, J4 Conn_01x01, K1 J104D2C12VDC.15S, K2 J104D2C12VDC.15S, K3 J104D2C12VDC.15S, K4 J104D2C12VDC.15S

Commit message: Add placeholders for JLC order number.
Other:
- board text added: "JLCJLCJLCJLC"
Changed lines of the file:
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@@
   (gr_line (start 173.99 63.5) (end 173.99 137.16)
     (stroke (width 0.1) (type default)) (layer "Edge.Cuts"))
+  (gr_text "JLCJLCJLCJLC" (at 172.72 135.89) (layer "B.SilkS")
+    (effects (font (size 1 1) (thickness 0.15)) (justify left bottom mirror))
+  )
   (gr_text "in 0" (at 107.95 99.06) (layer "F.SilkS")
     (effects (font (size 3 3) (thickness 0.6) bold) (justify left bottom))

Commit message: Add a "title" label to all parts.
Other:
- board text added: "vis vitalis eight-way mux"
Changed lines of the file:
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@@
   (gr_line (start 173.99 63.5) (end 173.99 137.16)
     (stroke (width 0.1) (type default)) (layer "Edge.Cuts"))
-  (gr_text "JLCJLCJLCJLC" (at 172.72 135.89) (layer "B.SilkS")
+  (gr_text "vis vitalis\neight-way mux" (at 171.196 134.366) (layer "B.SilkS")
+    (effects (font (size 3 3) (thickness 0.6) bold) (justify left bottom mirror))
+  )
+  (gr_text "JLCJLCJLCJLC" (at 107.95 125.73 90) (layer "B.SilkS")
     (effects (font (size 1 1) (thickness 0.15)) (justify left bottom mirror))
   )
