File: new-parts/add/add.kicad_pcb (KiCad board)
At the start: 2 copper layers, 97.8 x 125.7 mm, 30 parts, among them J1 BHR-10-VUA, J2 BHR-10-VUA, J3 BHR-10-VUA, J4 BHR-10-VUA, J5 Conn_01x02, J6 Conn_01x02, K1 J104D2C12VDC.15S, K10 J104D2C12VDC.15S, K11 J104D2C12VDC.15S, K12 J104D2C12VDC.15S, K13 J104D2C12VDC.15S, K14 J104D2C12VDC.15S, K15 J104D2C12VDC.15S, K16 J104D2C12VDC.15S, K2 J104D2C12VDC.15S, K3 J104D2C12VDC.15S, K4 J104D2C12VDC.15S, K5 J104D2C12VDC.15S, K6 J104D2C12VDC.15S, K7 J104D2C12VDC.15S, K8 J104D2C12VDC.15S, K9 J104D2C12VDC.15S

Commit message: Add placeholders for JLC order number.
Other:
- board text added: "JLCJLCJLCJLC"
Changed lines of the file:
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@@
   (gr_line (start 133.35 27.94) (end 133.35 153.67)
     (stroke (width 0.1) (type default)) (layer "Edge.Cuts"))
+  (gr_text "JLCJLCJLCJLC" (at 131.826 152.146) (layer "B.SilkS")
+    (effects (font (size 1 1) (thickness 0.15)) (justify left bottom mirror))
+  )
   (gr_text "A in" (at 41.91 64.77) (layer "F.SilkS")
     (effects (font (size 3 3) (thickness 0.6) bold) (justify left bottom))

Commit message: Add a "title" label to all parts.
Other:
- board text added: "vis vitalis adder"
Changed lines of the file:
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@@
     (effects (font (size 1 1) (thickness 0.15)) (justify left bottom mirror))
+  )
+  (gr_text "vis vitalis\nadder" (at 122.428 138.176 -90) (layer "B.SilkS")
+    (effects (font (size 3 3) (thickness 0.6) bold) (justify left bottom mirror))
   )
   (gr_text "A in" (at 41.91 64.77) (layer "F.SilkS")
