File: new-parts/add/add.kicad_pcb (KiCad board)
At the start: 2 copper layers, 97.8 x 125.7 mm, 30 parts, among them J1 BHR-10-VUA, J2 BHR-10-VUA, J3 BHR-10-VUA, J4 BHR-10-VUA, J5 Conn_01x02, J6 Conn_01x02, K1 J104D2C12VDC.15S, K10 J104D2C12VDC.15S, K11 J104D2C12VDC.15S, K12 J104D2C12VDC.15S, K13 J104D2C12VDC.15S, K14 J104D2C12VDC.15S, K15 J104D2C12VDC.15S, K16 J104D2C12VDC.15S, K2 J104D2C12VDC.15S, K3 J104D2C12VDC.15S, K4 J104D2C12VDC.15S, K5 J104D2C12VDC.15S, K6 J104D2C12VDC.15S, K7 J104D2C12VDC.15S, K8 J104D2C12VDC.15S, K9 J104D2C12VDC.15S

Commit message: Add signatures to some boards.
Other:
- board text added: "github.com/fread/visvitalis"
Changed lines of the file:
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@@
 		)
 	)
+	(gr_poly
+		(pts
+			(xy 39.499776 149.018686) (xy 37.345208 149.018686) (xy 37.345208 149.859999) (xy 38.904885 149.859999)
+			(xy 37.543302 151.221571) (xy 38.138205 151.816474) (xy 39.499778 150.454884) (xy 39.499778 152.014569)
+			(xy 40.34108 152.014569) (xy 40.34108 149.86) (xy 42.49561 149.86) (xy 42.49561 149.018687) (xy 40.935955 149.018687)
+			(xy 41.411992 148.542646) (xy 41.511089 148.448403) (xy 41.613658 148.360239) (xy 41.719467 148.278156)
+			(xy 41.828285 148.202153) (xy 41.93988 148.13223) (xy 42.054021 148.068387) (xy 42.170477 148.010625)
+			(xy 42.289015 147.958943) (xy 42.409406 147.913341) (xy 42.531416 147.87382) (xy 42.654815 147.840378)
+			(xy 42.779371 147.813017) (xy 42.904853 147.791736) (xy 43.03103 147.776536) (xy 43.157669 147.767415)
+			(xy 43.28454 147.764375) (xy 43.41141 147.767415) (xy 43.53805 147.776536) (xy 43.664226 147.791736)
+			(xy 43.789708 147.813017) (xy 43.914264 147.840378) (xy 44.037663 147.87382) (xy 44.159674 147.913341)
+			(xy 44.280064 147.958943) (xy 44.398603 148.010625) (xy 44.515058 148.068387) (xy 44.629199 148.13223)
+			(xy 44.740794 148.202153) (xy 44.849612 148.278156) (xy 44.955421 148.360239) (xy 45.05799 148.448403)
+			(xy 45.157087 148.542646) (xy 45.633127 149.018687) (xy 44.07347 149.018687) (xy 44.07347 149.86)
+			(xy 46.228 149.86) (xy 46.228 152.014569) (xy 47.069303 152.014569) (xy 47.069303 150.454864) (xy 48.430913 151.816474)
+			(xy 49.025777 151.221572) (xy 47.664214 149.86) (xy 49.223871 149.86) (xy 49.223871 149.018687) (xy 47.069303 149.018687)
+			(xy 47.069303 146.864157) (xy 46.227999 146.864155) (xy 46.227999 148.423784) (xy 45.751987 147.947774)
+			(xy 45.622103 147.82433) (xy 45.48751 147.708851) (xy 45.348522 147.601335) (xy 45.205452 147.501782)
+			(xy 45.058615 147.410193) (xy 44.908325 147.326568) (xy 44.754896 147.250907) (xy 44.598641 147.183209)
+			(xy 44.439874 147.123476) (xy 44.27891 147.071707) (xy 44.116063 147.027902) (xy 43.951645 146.992062)
+			(xy 43.785972 146.964186) (xy 43.619357 146.944274) (xy 43.452115 146.932327) (xy 43.284558 146.928345)
+			(xy 43.117002 146.932327) (xy 42.949759 146.944274) (xy 42.783144 146.964186) (xy 42.617471 146.992062)
+			(xy 42.453054 147.027902) (xy 42.290206 147.071707) (xy 42.129242 147.123476) (xy 41.970475 147.183209)
+			(xy 41.81422 147.250907) (xy 41.660791 147.326568) (xy 41.5105 147.410193) (xy 41.363663 147.501782)
+			(xy 41.220594 147.601335) (xy 41.081606 147.708851) (xy 40.947012 147.82433) (xy 40.817128 147.947774)
+			(xy 40.341079 148.423823) (xy 40.341079 146.864155) (xy 39.499776 146.864155)
+		)
+		(stroke
+			(width -0.000001)
+			(type solid)
+		)
+		(fill solid)
+		(layer "B.SilkS")
+	)
 	(gr_line
 		(start 35.56 153.67)
@@
 		)
 	)
+	(gr_text "github.com/fread/visvitalis"
+		(at 50.8 149.352 0)
+		(layer "B.SilkS")
+		(effects
+			(font
+				(size 1.5 1.5)
+				(thickness 0.3)
+				(bold yes)
+			)
+			(justify right mirror)
+		)
+	)
 	(gr_text "vis vitalis\nadder"
 		(at 122.428 138.176 -90)
@@
 		)
 	)
+	(group ""
+		(members "ce7dc386-b1bc-4a7d-a97a-d4a5271deaf0")
+	)
 )
