File: new-parts/jnc/jnc.kicad_pcb (KiCad board)
At the start: 2 copper layers, 20.3 x 97.8 mm, 4 parts, among them J1 BHR-10-VUA, J2 BHR-10-VUA, J3 BHR-10-VUA, J4 BHR-10-VUA

Commit message: Add placeholders for JLC order number.
Other:
- board text added: "JLCJLCJLCJLC"
Changed lines of the file:
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@@
   (gr_line (start 144.78 53.34) (end 144.78 151.13)
     (stroke (width 0.1) (type default)) (layer "Edge.Cuts"))
+  (gr_text "JLCJLCJLCJLC" (at 143.256 149.606) (layer "B.SilkS")
+    (effects (font (size 1 1) (thickness 0.15)) (justify left bottom mirror))
+  )
   (segment (start 133.35 85.09) (end 127 85.09) (width 0.4) (layer "F.Cu") (net 1))
   (segment (start 133.35 109.22) (end 127 109.22) (width 0.4) (layer "F.Cu") (net 1))

Commit message: Add a "title" label to all parts.
Other:
- board text added: "junction"
- board text added: "vis"
- board text added: "vitalis"
Changed lines of the file:
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@@
   (gr_line (start 144.78 53.34) (end 144.78 151.13)
     (stroke (width 0.1) (type default)) (layer "Edge.Cuts"))
+  (gr_text "junction" (at 139.7 83.82 270) (layer "B.SilkS")
+    (effects (font (size 3 3) (thickness 0.6) bold) (justify left bottom mirror))
+  )
+  (gr_text "vitalis" (at 139.7 108.204 270) (layer "B.SilkS")
+    (effects (font (size 3 3) (thickness 0.6) bold) (justify left bottom mirror))
+  )
   (gr_text "JLCJLCJLCJLC" (at 143.256 149.606) (layer "B.SilkS")
     (effects (font (size 1 1) (thickness 0.15)) (justify left bottom mirror))
   )
+  (gr_text "vis" (at 139.7 121.666 270) (layer "B.SilkS")
+    (effects (font (size 3 3) (thickness 0.6) bold) (justify left bottom mirror))
+  )
   (segment (start 133.35 85.09) (end 127 85.09) (width 0.4) (layer "F.Cu") (net 1))
