File: new-parts/nor/nor.kicad_pcb (KiCad board)
At the start: 2 copper layers, 78.7 x 106.7 mm, 35 parts, among them J1 BHR-10-VUA, J2 BHR-10-VUA, J3 BHR-10-VUA, K1 J104D2C12VDC.15S, K2 J104D2C12VDC.15S, K3 J104D2C12VDC.15S, K4 J104D2C12VDC.15S, K5 J104D2C12VDC.15S, K6 J104D2C12VDC.15S, K7 J104D2C12VDC.15S, K8 J104D2C12VDC.15S

Commit message: Add placeholders for JLC order number.
Other:
- board text added: "JLCJLCJLCJLC"
Changed lines of the file:
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@@
   (gr_line (start 185.42 40.64) (end 185.42 147.32)
     (stroke (width 0.1) (type default)) (layer "Edge.Cuts"))
+  (gr_text "JLCJLCJLCJLC" (at 183.896 145.796) (layer "B.SilkS")
+    (effects (font (size 1 1) (thickness 0.15)) (justify left bottom mirror))
+  )
   (gr_text "B in" (at 109.22 95.25) (layer "F.SilkS")
     (effects (font (size 3 3) (thickness 0.6) bold) (justify left bottom))

Commit message: Add a "title" label to all parts.
Other:
- board text added: "vis vitalis nor gate"
Changed lines of the file:
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@@
     (effects (font (size 1 1) (thickness 0.15)) (justify left bottom mirror))
+  )
+  (gr_text "vis vitalis\nnor gate" (at 177.8 142.24 270) (layer "B.SilkS")
+    (effects (font (size 3 3) (thickness 0.6) bold) (justify left mirror))
   )
   (gr_text "B in" (at 109.22 95.25) (layer "F.SilkS")
