File: new-parts/or/or.kicad_pcb (KiCad board)
At the start: 2 copper layers, 44.5 x 63.5 mm, 19 parts, among them J1 BHR-10-VUA, J2 BHR-10-VUA, J3 BHR-10-VUA

Commit message: Add placeholders for JLC order number.
Other:
- board text added: "JLCJLCJLCJLC"
Changed lines of the file:
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@@
   (gr_line (start 152.4 63.5) (end 152.4 127)
     (stroke (width 0.1) (type default)) (layer "Edge.Cuts"))
+  (gr_text "JLCJLCJLCJLC" (at 150.876 125.476) (layer "B.SilkS")
+    (effects (font (size 1 1) (thickness 0.15)) (justify left bottom mirror))
+  )
   (gr_text "A in" (at 110.49 69.85) (layer "F.SilkS")
     (effects (font (size 3 3) (thickness 0.6) bold) (justify left bottom))

Commit message: Add a "title" label to all parts.
Other:
- board text added: "vis vitalis or gate"
Changed lines of the file:
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@@
   (gr_line (start 152.4 63.5) (end 152.4 127)
     (stroke (width 0.1) (type default)) (layer "Edge.Cuts"))
+  (gr_text "vis vitalis\nor gate" (at 140.97 87.63 -90) (layer "B.SilkS")
+    (effects (font (size 3 3) (thickness 0.6) bold) (justify left bottom mirror))
+  )
   (gr_text "JLCJLCJLCJLC" (at 150.876 125.476) (layer "B.SilkS")
     (effects (font (size 1 1) (thickness 0.15)) (justify left bottom mirror))
