File: new-parts/disp/disp.kicad_pcb (KiCad board)
At the start: 2 copper layers, 76.2 x 39.4 mm, 18 parts, among them J1 BHR-10-VUA, J2 BHR-10-VUA

Commit message: Changes made by JLCPCB fabrication plugin.
Other:
- board size 76.2 x 39.4 mm -> 68.6 x 39.4 mm
Changed lines of the file:
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@@
 	(setup
 		(pad_to_mask_clearance 0.038)
-		(solder_mask_min_width 0.1)
 		(allow_soldermask_bridges_in_footprints no)
 		(pcbplotparams
@@
 		(tags "resistor handsolder")
 		(property "Reference" "R3"
-			(at 0 -1.65 90)
+			(at 3.175 0 90)
 			(layer "F.SilkS")
 			(effects
@@
 		(tags "resistor handsolder")
 		(property "Reference" "R8"
-			(at 0 -1.65 90)
+			(at 3.175 0 90)
 			(layer "F.SilkS")
 			(effects
@@
 		(tags "resistor handsolder")
 		(property "Reference" "R2"
-			(at 0 -1.65 90)
+			(at 3.175 0 90)
 			(layer "F.SilkS")
 			(effects
@@
 		(tags "resistor handsolder")
 		(property "Reference" "R4"
-			(at 0 -1.65 90)
+			(at 3.175 0 90)
 			(layer "F.SilkS")
 			(effects
@@
 		(tags "resistor handsolder")
 		(property "Reference" "R7"
-			(at 0 -1.65 90)
+			(at 3.175 0 90)
 			(layer "F.SilkS")
 			(effects
@@
 		(tags "resistor handsolder")
 		(property "Reference" "R1"
-			(at 0 -1.65 90)
+			(at 3.175 0 90)
 			(layer "F.SilkS")
 			(effects
@@
 		(tags "resistor handsolder")
 		(property "Reference" "R6"
-			(at 0 -1.65 90)
+			(at 3.175 0 90)
 			(layer "F.SilkS")
 			(effects
@@
 		(tags "resistor handsolder")
 		(property "Reference" "R5"
-			(at 0 -1.65 90)
+			(at 3.175 0 90)
 			(layer "F.SilkS")
 			(effects
@@
 	)
 	(gr_line
-		(start 200.66 127)
-		(end 124.46 127)
+		(start 198.12 127)
+		(end 129.54 127)
 		(stroke
 			(width 0.1)
@@
 	)
 	(gr_line
-		(start 124.46 87.63)
-		(end 200.66 87.63)
+		(start 129.54 87.63)
+		(end 198.12 87.63)
 		(stroke
 			(width 0.1)
@@
 	)
 	(gr_line
-		(start 124.46 127)
-		(end 124.46 87.63)
+		(start 129.54 127)
+		(end 129.54 87.63)
 		(stroke
 			(width 0.1)
@@
 	)
 	(gr_line
-		(start 200.66 87.63)
-		(end 200.66 127)
+		(start 198.12 87.63)
+		(end 198.12 127)
 		(stroke
 			(width 0.1)
@@
 		(layer "Dwgs.User")
 		(pts
-			(xy 124.46 129.54) (xy 200.66 129.54)
+			(xy 127 129.54) (xy 198.12 129.54)
 		)
 		(height 2.54)
-		(gr_text "76.2000 mm"
+		(gr_text "71.1200 mm"
 			(at 162.56 130.93 0)
 			(layer "Dwgs.User")
@@
 		(layer "Dwgs.User")
 		(pts
-			(xy 121.92 87.63) (xy 121.92 127)
+			(xy 127 87.63) (xy 127 127)
 		)
 		(height 2.54)
 		(gr_text "39.3700 mm"
-			(at 118.23 107.315 90)
+			(at 123.31 107.315 90)
 			(layer "Dwgs.User")
 			(effects
@@
 		(polygon
 			(pts
-				(xy 123.19 86.36) (xy 201.93 86.36) (xy 201.93 128.27) (xy 123.19 128.27)
+				(xy 128.27 86.36) (xy 199.39 86.36) (xy 199.39 128.27) (xy 128.27 128.27)
 			)
 		)
@@
 		(polygon
 			(pts
-				(xy 123.19 86.36) (xy 201.93 86.36) (xy 201.93 128.27) (xy 123.19 128.27)
+				(xy 128.27 86.36) (xy 199.39 86.36) (xy 199.39 128.27) (xy 128.27 128.27)
 			)
 		)
