File: new-parts/reg/reg.kicad_pcb (KiCad board)
At the start: 2 copper layers, 104.1 x 113 mm, 51 parts, among them J1 BHR-10-VUA, J2 BHR-10-VUA, J3 BHR-10-VUA, J4 BHR-10-VUA, J5 Conn_01x02, J6 Conn_02x02_Odd_Even, K1 J104D2C12VDC.15S, K10 J104D2C12VDC.15S, K11 J104D2C12VDC.15S, K12 J104D2C12VDC.15S, K2 J104D2C12VDC.15S, K3 J104D2C12VDC.15S, K4 J104D2C12VDC.15S, K5 J104D2C12VDC.15S, K6 J104D2C12VDC.15S, K7 J104D2C12VDC.15S, K8 J104D2C12VDC.15S, K9 J104D2C12VDC.15S

Commit message: Add signatures to some boards.
Other:
- board text added: "github.com/fread/visvitalis"
Changed lines of the file:
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@@
 		)
+	)
+	(gr_poly
+		(pts
+			(xy 113.03 37.714531) (xy 110.875432 37.714531) (xy 110.875432 38.555844) (xy 112.435109 38.555844)
+			(xy 111.073526 39.917416) (xy 111.668429 40.512319) (xy 113.030002 39.150729) (xy 113.030002 40.710414)
+			(xy 113.871304 40.710414) (xy 113.871304 38.555845) (xy 116.025834 38.555845) (xy 116.025834 37.714532)
+			(xy 114.466179 37.714532) (xy 114.942216 37.238491) (xy 115.041313 37.144248) (xy 115.143882 37.056084)
+			(xy 115.249691 36.974001) (xy 115.358509 36.897998) (xy 115.470104 36.828075) (xy 115.584245 36.764232)
+			(xy 115.700701 36.70647) (xy 115.819239 36.654788) (xy 115.93963 36.609186) (xy 116.06164 36.569665)
+			(xy 116.185039 36.536223) (xy 116.309595 36.508862) (xy 116.435077 36.487581) (xy 116.561254 36.472381)
+			(xy 116.687893 36.46326) (xy 116.814764 36.46022) (xy 116.941634 36.46326) (xy 117.068274 36.472381)
+			(xy 117.19445 36.487581) (xy 117.319932 36.508862) (xy 117.444488 36.536223) (xy 117.567887 36.569665)
+			(xy 117.689898 36.609186) (xy 117.810288 36.654788) (xy 117.928827 36.70647) (xy 118.045282 36.764232)
+			(xy 118.159423 36.828075) (xy 118.271018 36.897998) (xy 118.379836 36.974001) (xy 118.485645 37.056084)
+			(xy 118.588214 37.144248) (xy 118.687311 37.238491) (xy 119.163351 37.714532) (xy 117.603694 37.714532)
+			(xy 117.603694 38.555845) (xy 119.758224 38.555845) (xy 119.758224 40.710414) (xy 120.599527 40.710414)
+			(xy 120.599527 39.150709) (xy 121.961137 40.512319) (xy 122.556001 39.917417) (xy 121.194438 38.555845)
+			(xy 122.754095 38.555845) (xy 122.754095 37.714532) (xy 120.599527 37.714532) (xy 120.599527 35.560002)
+			(xy 119.758223 35.56) (xy 119.758223 37.119629) (xy 119.282211 36.643619) (xy 119.152327 36.520175)
+			(xy 119.017734 36.404696) (xy 118.878746 36.29718) (xy 118.735676 36.197627) (xy 118.588839 36.106038)
+			(xy 118.438549 36.022413) (xy 118.28512 35.946752) (xy 118.128865 35.879054) (xy 117.970098 35.819321)
+			(xy 117.809134 35.767552) (xy 117.646287 35.723747) (xy 117.481869 35.687907) (xy 117.316196 35.660031)
+			(xy 117.149581 35.640119) (xy 116.982339 35.628172) (xy 116.814782 35.62419) (xy 116.647226 35.628172)
+			(xy 116.479983 35.640119) (xy 116.313368 35.660031) (xy 116.147695 35.687907) (xy 115.983278 35.723747)
+			(xy 115.82043 35.767552) (xy 115.659466 35.819321) (xy 115.500699 35.879054) (xy 115.344444 35.946752)
+			(xy 115.191015 36.022413) (xy 115.040724 36.106038) (xy 114.893887 36.197627) (xy 114.750818 36.29718)
+			(xy 114.61183 36.404696) (xy 114.477236 36.520175) (xy 114.347352 36.643619) (xy 113.871303 37.119668)
+			(xy 113.871303 35.56) (xy 113.03 35.56)
+		)
+		(stroke
+			(width -0.000001)
+			(type solid)
+		)
+		(fill solid)
+		(layer "B.SilkS")
 	)
 	(gr_line
@@
 	)
 	(gr_text "JLCJLCJLCJLC"
-		(at 201.676 143.256 0)
+		(at 100.33 143.51 0)
 		(layer "B.SilkS")
 		(effects
@@
 				(thickness 0.15)
 			)
-			(justify left bottom mirror)
+			(justify right bottom mirror)
 		)
 	)
+	(gr_text "github.com/fread/visvitalis"
+		(at 123.952 38.1 0)
+		(layer "B.SilkS")
+		(effects
+			(font
+				(size 1.5 1.5)
+				(thickness 0.3)
+				(bold yes)
+			)
+			(justify right mirror)
+		)
+	)
 	(gr_text "vis vitalis\nregister"
-		(at 194.31 139.7 270)
+		(at 200.152 35.306 0)
 		(layer "B.SilkS")
 		(effects
@@
 				(bold yes)
 			)
-			(justify left mirror)
+			(justify left top mirror)
 		)
 	)
@@
 		)
 	)
+	(group ""
+		(members "75dad89a-3df2-4bf1-9622-ab0f10d6a406")
+	)
 )
